File: Leah/DriverDisplay.kicad_pcb (KiCad board)
At the start: 2 copper layers, 7 parts, among them U1 MCP2551-I-SN, U2 V7805-500

Commit message: added kicad designs
Parts:
- added C2: 10u, Capacitor_SMD:C_0805_2012Metric_Pad1.15x1.40mm_HandSolder, F.Cu at (167.6, 93.0)
- added C3: 22u, Capacitor_SMD:C_0805_2012Metric_Pad1.15x1.40mm_HandSolder, F.Cu at (161.3, 90.2)
- added C5: .1u, Capacitor_SMD:C_0805_2012Metric_Pad1.15x1.40mm_HandSolder, F.Cu at (94.0, 92.7)
- added C6: .1u, Capacitor_SMD:C_0805_2012Metric_Pad1.15x1.40mm_HandSolder, F.Cu at (94.2, 81.3)
- added H1: MountingHole, MountingHole:MountingHole_3.2mm_M3, F.Cu at (83.8, 71.1)
- added H2: MountingHole, MountingHole:MountingHole_3.2mm_M3, F.Cu at (168.9, 71.1)
- added H3: MountingHole, MountingHole:MountingHole_3.2mm_M3, F.Cu at (168.9, 104.1)
- added H4: MountingHole, MountingHole:MountingHole_3.2mm_M3, F.Cu at (83.8, 104.1)
- added J1: GLV/CAN, Connector_JST:JST_PH_S4B-PH-SM4-TB_1x04-1MP_P2.00mm_Horizontal, F.Cu at (180.3, 99.3)
- added J2: Display, Connector_JST:JST_PH_S8B-PH-SM4-TB_1x08-1MP_P2.00mm_Horizontal, F.Cu at (180.3, 78.7)
- added R10: 750, Resistor_SMD:R_0805_2012Metric_Pad1.15x1.40mm_HandSolder, F.Cu at (80.0, 99.1)
- added R11: 1K, Resistor_SMD:R_0805_2012Metric_Pad1.15x1.40mm_HandSolder, F.Cu at (86.4, 81.3)
- added R2: 1K, Resistor_SMD:R_0805_2012Metric_Pad1.15x1.40mm_HandSolder, F.Cu at (124.5, 85.1)
- added R3: 120, Resistor_SMD:R_0805_2012Metric_Pad1.15x1.40mm_HandSolder, F.Cu at (129.5, 90.2)
- added R4: 100k, Resistor_SMD:R_0805_2012Metric_Pad1.15x1.40mm_HandSolder, F.Cu at (90.2, 88.9)
- added R5: 1K, Resistor_SMD:R_0805_2012Metric_Pad1.15x1.40mm_HandSolder, F.Cu at (87.6, 92.7)
- added R6: 100k, Resistor_SMD:R_0805_2012Metric_Pad1.15x1.40mm_HandSolder, F.Cu at (90.2, 85.1)
- added R7: 68, Resistor_SMD:R_0805_2012Metric_Pad1.15x1.40mm_HandSolder, F.Cu at (80.0, 73.7)
- added R8: 750, Resistor_SMD:R_0805_2012Metric_Pad1.15x1.40mm_HandSolder, F.Cu at (80.0, 77.5)
- added R9: 68, Resistor_SMD:R_0805_2012Metric_Pad1.15x1.40mm_HandSolder, F.Cu at (80.0, 102.9)
- moved D4 132.1 mm to (71.1, 100.3)
- moved BTN1 131.7 mm to (54.6, 87.6)
- moved D3 128.1 mm to (71.1, 74.9)
- moved BTN2 114.1 mm to (72.4, 87.6)
- moved U1 67.5 mm to (129.5, 83.8), turned to 270 degrees
- moved ESP321 37.7 mm to (151.1, 99.1), turned to 90 degrees
- moved U2 16.9 mm to (160.0, 97.8), turned to 90 degrees
Connections:
- BTN1 pad 1: Net-(BTN1-Pad1) -> /ESP_GND
- BTN1 pad 2: Net-(BTN1-Pad2) -> /BUTTON1
- BTN2 pad 1: Net-(BTN2-Pad1) -> /ESP_GND
- BTN2 pad 2: Net-(BTN2-Pad2) -> /BUTTON2
- ESP321 pad 20: Net-(ESP321-Pad20) -> /CANTX
- ESP321 pad 23: Net-(ESP321-Pad23) -> /CANRX
- ESP321 pad 24: /~R2 -> Net-(ESP321-Pad24)
- ESP321 pad 25: /~G2 -> Net-(ESP321-Pad25)
- ESP321 pad 4: /BUTTON1 -> /ESP_BUTTON1
- ESP321 pad 5: /BUTTON2 -> /ESP_BUTTON2
- ESP321 pad 8: Net-(ESP321-Pad8) -> /~R2
- ESP321 pad 9: Net-(ESP321-Pad9) -> /~G2
Routing:
- net /ESP_3V3: track 0.00 -> 189.8 mm
- net /ESP_GND: track 0.00 -> 187.4 mm
- net /GLV_RTN: track 0.00 -> 113.5 mm
- net /CLK: track 0.00 -> 84.3 mm
- net /DIN: track 0.00 -> 76.9 mm
- net /DC: track 0.00 -> 72.5 mm, vias 0 -> 1
- net /RST: track 0.00 -> 70.9 mm
- net /CAN_L: track 0.00 -> 64.4 mm
- net /~R1: track 0.00 -> 59.1 mm
- net /CAN_H: track 0.00 -> 56.0 mm
- net /ESP_BUTTON2: track 0.00 -> 54.0 mm
- net /BUSY: track 0.00 -> 53.1 mm
- net /~G2: track 0.00 -> 48.8 mm
- net /~G1: track 0.00 -> 48.1 mm
- net /CS: track 0.00 -> 46.5 mm
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