File: Leah/DriverDisplay.sch (KiCad schematic (older format))
At the start: 17 parts, among them J1 GLV/CAN, J2 Display, U1 MCP2551-I-SN, U2 V7805-500

Commit message: added kicad designs
Parts:
- removed C1: 0.1u, symbol Device:C
- removed R1: 1k, symbol Device:R
- added C5, C6: .1u, Capacitor_SMD:C_0805_2012Metric_Pad1.15x1.40mm_HandSolder, symbol Device:C
- added H1, H2, H3, H4: MountingHole, MountingHole:MountingHole_3.2mm_M3, symbol Mechanical:MountingHole
- added R11, R2, R5: 1K, Resistor_SMD:R_0805_2012Metric_Pad1.15x1.40mm_HandSolder, symbol Device:R
- added R3: 120, Resistor_SMD:R_0805_2012Metric_Pad1.15x1.40mm_HandSolder, symbol Device:R
- added R4, R6: 100k, Resistor_SMD:R_0805_2012Metric_Pad1.15x1.40mm_HandSolder, symbol Device:R
- C2, C3: footprint (none) -> Capacitor_SMD:C_0805_2012Metric_Pad1.15x1.40mm_HandSolder
- J1: footprint (none) -> Connector_JST:JST_PH_S4B-PH-SM4-TB_1x04-1MP_P2.00mm_Horizontal; symbol Connector_Generic:Conn_01x06 -> Connector_Generic:Conn_01x04
- J2: footprint (none) -> Connector_JST:JST_PH_S8B-PH-SM4-TB_1x08-1MP_P2.00mm_Horizontal
- R10, R8: value R -> 750; footprint (none) -> Resistor_SMD:R_0805_2012Metric_Pad1.15x1.40mm_HandSolder
- R7, R9: value R -> 68; footprint (none) -> Resistor_SMD:R_0805_2012Metric_Pad1.15x1.40mm_HandSolder
Connections:
- net CAN_SHIELD is gone; now on net GLV_24V: J1.3 (Pin_3)
- net BUTTON1: now also BTN1.2, R5.2; no longer ESP321.4 (GPIO34)
- net BUTTON2: now also BTN2.2, R11.2; no longer ESP321.5 (GPIO35)
- net CANRX: now also ESP321.23 (GPIO5)
- net CANTX: now also ESP321.20 (GPIO4)
- net CAN_H: now also R3.1
- net CAN_L: now also R3.2
- net ESP_3V3: now also R4.2, R6.2
- net ESP_GND: now also BTN1.1, BTN2.1
- net GLV_24V: no longer J1.4 (Pin_4)
- net GLV_RTN: now also J1.4 (Pin_4), C5.2, C6.2, R2.1; no longer J1.5 (Pin_5)
- net ~G2: now also ESP321.9 (GPIO26); no longer ESP321.25 (GPIO19)
- net ~R2: now also ESP321.8 (GPIO25); no longer ESP321.24 (GPIO18)
- net at U1.8 (Rs): now also R2.2
- removed net CHS_GND: J1.6 (Pin_6)
- new net ESP_BUTTON1: C5.1, ESP321.4 (GPIO34), R4.1, R5.1
- new net ESP_BUTTON2: C6.1, ESP321.5 (GPIO35), R11.1, R6.1
Other:
- note added: "Do not populate 120ohm resistor. Footprint is left open for debugging."
- moved on the sheet: BTN1, BTN2, C2, C3, U1, U2
