File: Leah/DriverDisplay2.kicad_pcb (KiCad board)
At the start: 2 copper layers, 30 parts, among them J1 GLV/CAN, J2 Display, U1 MCP2551-I-SN, U2 V7805-500, U3 V7809-500

Commit message: updated dashboard 2.0
Routing:
- net /ESP_GND: track 0.00 -> 184.3 mm, vias 0 -> 1
- net /ESP_3V3: track 0.00 -> 125.0 mm, vias 0 -> 4
- net /DC: track 0.00 -> 85.5 mm, vias 0 -> 3
- net /RST: track 0.00 -> 73.6 mm, vias 0 -> 3
- net /~R1: track 0.00 -> 73.3 mm, vias 0 -> 1
- net /GLV_RTN: track 89.9 -> 160.1 mm, vias 2 -> 4
- net /CAN_L: track 4.04 -> 72.0 mm, vias 0 -> 2
- net /CAN_H: track 4.04 -> 71.7 mm, vias 0 -> 2
- net /~G1: track 0.00 -> 60.6 mm, vias 0 -> 1
- net /BUSY: track 0.00 -> 60.1 mm, vias 0 -> 3
- net /CLK: track 0.00 -> 56.8 mm, vias 0 -> 1
- net /CS: track 0.00 -> 55.3 mm, vias 0 -> 2
- net /BUTTON1: track 0.00 -> 49.9 mm, vias 0 -> 1
- net /DIN: track 0.00 -> 49.7 mm, vias 0 -> 1
- net /~G2: track 0.00 -> 43.0 mm, vias 0 -> 2
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