File: Leah/DriverDisplay4.kicad_pcb (KiCad board)
At the start: 2 copper layers, 126.8 x 42.3 mm, 34 parts, among them J1 GLV/CAN, J2 Display, U1 MCP2551-I-SN, U2 L78L05CD13TR, U3 L78L09CD13TR, U4 2.9epaper

Commit message: v4 board
Routing:
- net /BUTTON1: track 52.5 -> 39.0 mm
- net Net-(D4-Pad1): track 7.20 -> 19.0 mm
- net /BUTTON2: track 29.0 -> 32.2 mm
- net /ESP_GND: track 157.6 -> 160.4 mm
