File: Leah/DriverDisplay2.sch (KiCad schematic (older format))
At the start: 23 parts, among them J1 GLV/CAN, J2 Display, U1 MCP2551-I-SN, U2 V7805-500

Commit message: added kicad designs
Parts:
- added C1, C4: 10u, Capacitor_SMD:C_0805_2012Metric_Pad1.15x1.40mm_HandSolder, symbol Device:C
- added H1, H2, H3, H4: MountingHole, MountingHole:MountingHole_3.2mm_M3, symbol Mechanical:MountingHole
- added U3: V7809-500, Lafayette_Electric_Car_Footprints:VX7805-500, symbol Lafayette_Electric_Car_Internals:V7809-500
Connections:
- net labels added: GLV_9V
- net labels removed: CANH, CANL
- wire segments 86 -> 100
Other:
- note added: "Do not populate 120ohm resistor. Footprint is left open for debugging."
- moved on the sheet: C2, C3, U2
Changed lines of the file:
@@
 L Lafayette_Electric_Car_Internals:V7805-500 U2
 U 1 1 5DD5D737
-P 3350 1600
-F 0 "U2" H 3600 1767 50  0000 C CNN
-F 1 "V7805-500" H 3600 1676 50  0000 C CNN
-F 2 "Lafayette_Electric_Car_Footprints:VX7805-500" H 2850 1700 50  0001 C CNN
-F 3 "https://www.cui.com/product/resource/v78-500.pdf" H 2850 1700 50  0001 C CNN
-	1    3350 1600
+P 3250 1000
+F 0 "U2" H 3500 1167 50  0000 C CNN
+F 1 "V7805-500" H 3500 1076 50  0000 C CNN
+F 2 "Lafayette_Electric_Car_Footprints:VX7805-500" H 2750 1100 50  0001 C CNN
+F 3 "https://www.cui.com/product/resource/v78-500.pdf" H 2750 1100 50  0001 C CNN
+	1    3250 1000
 	1    0    0    -1
 $EndComp
@@
 L Device:C C3
 U 1 1 5DD5DF3D
-P 4100 1950
-F 0 "C3" H 4215 1996 50  0000 L CNN
-F 1 "22u" H 4215 1905 50  0000 L CNN
-F 2 "Capacitor_SMD:C_0805_2012Metric_Pad1.15x1.40mm_HandSolder" H 4138 1800 50  0001 C CNN
-F 3 "~" H 4100 1950 50  0001 C CNN
-	1    4100 1950
+P 4000 1350
+F 0 "C3" H 4115 1396 50  0000 L CNN
+F 1 "22u" H 4115 1305 50  0000 L CNN
+F 2 "Capacitor_SMD:C_0805_2012Metric_Pad1.15x1.40mm_HandSolder" H 4038 1200 50  0001 C CNN
+F 3 "~" H 4000 1350 50  0001 C CNN
+	1    4000 1350
 	1    0    0    -1
 $EndComp
@@
 L Device:C C2
 U 1 1 5DD5E24C
-P 3050 1950
-F 0 "C2" H 3165 1996 50  0000 L CNN
-F 1 "10u" H 3165 1905 50  0000 L CNN
-F 2 "Capacitor_SMD:C_0805_2012Metric_Pad1.15x1.40mm_HandSolder" H 3088 1800 50  0001 C CNN
-F 3 "~" H 3050 1950 50  0001 C CNN
-	1    3050 1950
+P 2950 1350
+F 0 "C2" H 3065 1396 50  0000 L CNN
+F 1 "10u" H 3065 1305 50  0000 L CNN
+F 2 "Capacitor_SMD:C_0805_2012Metric_Pad1.15x1.40mm_HandSolder" H 2988 1200 50  0001 C CNN
+F 3 "~" H 2950 1350 50  0001 C CNN
+	1    2950 1350
 	1    0    0    -1
 $EndComp
@@
 Wire Wire Line
 	1450 2900 1350 2900
-Text Label 2950 2200 2    50   ~ 0
-GLV_RTN
-Wire Wire Line
-	2950 2200 3050 2200
-Wire Wire Line
-	4100 2200 4100 2100
-Wire Wire Line
-	3600 2100 3600 2200
-Connection ~ 3600 2200
-Wire Wire Line
-	3600 2200 4100 2200
-Wire Wire Line
-	3050 2100 3050 2200
-Connection ~ 3050 2200
-Wire Wire Line
-	3050 2200 3600 2200
-Wire Wire Line
-	3050 1800 3050 1700
-Wire Wire Line
-	3050 1700 3250 1700
-Wire Wire Line
-	3950 1700 4100 1700
-Wire Wire Line
-	4100 1700 4100 1800
-Text Label 2950 1700 2    50   ~ 0
+Text Label 2850 1600 2    50   ~ 0
+GLV_RTN
+Wire Wire Line
+	2850 1600 2950 1600
+Wire Wire Line
+	4000 1600 4000 1500
+Wire Wire Line
+	3500 1500 3500 1600
+Connection ~ 3500 1600
+Wire Wire Line
+	3500 1600 4000 1600
+Wire Wire Line
+	2950 1500 2950 1600
+Connection ~ 2950 1600
+Wire Wire Line
+	2950 1600 3500 1600
+Wire Wire Line
+	2950 1200 2950 1100
+Wire Wire Line
+	2950 1100 3150 1100
+Wire Wire Line
+	3850 1100 4000 1100
+Wire Wire Line
+	4000 1100 4000 1200
+Text Label 2850 1100 2    50   ~ 0
 GLV_24V
 Wire Wire Line
-	2950 1700 3050 1700
-Connection ~ 3050 1700
-Text Label 4200 1700 0    50   ~ 0
+	2850 1100 2950 1100
+Connection ~ 2950 1100
+Text Label 4100 1100 0    50   ~ 0
 GLV_5V
 Wire Wire Line
-	4200 1700 4100 1700
-Connection ~ 4100 1700
+	4100 1100 4000 1100
+Connection ~ 4000 1100
 $Comp
 L Connector_Generic:Conn_01x08 J2
@@
 ~G1
 Wire Wire Line
-	6375 3950 6450 3950
-Text Label 6450 3950 0    50   ~ 0
+	4925 4150 4850 4150
+Text Label 4850 4150 2    50   ~ 0
+~G2
+Wire Wire Line
+	4925 4050 4850 4050
+Text Label 4850 4050 2    50   ~ 0
 ~R2
-Wire Wire Line
-	6375 3850 6450 3850
-Text Label 6450 3850 0    50   ~ 0
-~G2
 $Comp
 L Lafayette_Electric_Car_Internals:PushButton BTN2
@@
 Connection ~ 3550 5800
 Text Label 3750 5500 0    50   ~ 0
-CANH
+CAN_H
 Text Label 3750 5800 0    50   ~ 0
-CANL
+CAN_L
 $Comp
 L Device:C C5
@@
 Text Label 1800 5850 2    50   ~ 0
 GLV_RTN
+$Comp
+L Mechanical:MountingHole H1
+U 1 1 5E5587CE
+P 2800 3200
+F 0 "H1" H 2900 3246 50  0000 L CNN
+F 1 "MountingHole" H 2900 3155 50  0000 L CNN
+F 2 "MountingHole:MountingHole_3.2mm_M3" H 2800 3200 50  0001 C CNN
+F 3 "~" H 2800 3200 50  0001 C CNN
+	1    2800 3200
+	1    0    0    -1
+$EndComp
+$Comp
+L Mechanical:MountingHole H2
+U 1 1 5E55ADD8
+P 2800 3450
+F 0 "H2" H 2900 3496 50  0000 L CNN
+F 1 "MountingHole" H 2900 3405 50  0000 L CNN
+F 2 "MountingHole:MountingHole_3.2mm_M3" H 2800 3450 50  0001 C CNN
+F 3 "~" H 2800 3450 50  0001 C CNN
+	1    2800 3450
+	1    0    0    -1
+$EndComp
+$Comp
+L Mechanical:MountingHole H3
+U 1 1 5E55D975
+P 2800 3700
+F 0 "H3" H 2900 3746 50  0000 L CNN
+F 1 "MountingHole" H 2900 3655 50  0000 L CNN
+F 2 "MountingHole:MountingHole_3.2mm_M3" H 2800 3700 50  0001 C CNN
+F 3 "~" H 2800 3700 50  0001 C CNN
+	1    2800 3700
+	1    0    0    -1
+$EndComp
+$Comp
+L Mechanical:MountingHole H4
+U 1 1 5E560686
+P 2800 3950
+F 0 "H4" H 2900 3996 50  0000 L CNN
+F 1 "MountingHole" H 2900 3905 50  0000 L CNN
+F 2 "MountingHole:MountingHole_3.2mm_M3" H 2800 3950 50  0001 C CNN
+F 3 "~" H 2800 3950 50  0001 C CNN
+	1    2800 3950
+	1    0    0    -1
+$EndComp
+Text Notes 3450 6050 0    50   ~ 0
+Do not populate 120ohm resistor. Footprint is left open for debugging.
+$Comp
+L Lafayette_Electric_Car_Internals:V7809-500 U3
+U 1 1 5E5E366E
+P 3500 1900
+F 0 "U3" H 3500 1817 50  0000 C CNN
+F 1 "V7809-500" H 3500 1726 50  0000 C CNN
+F 2 "Lafayette_Electric_Car_Footprints:VX7805-500" H 3500 1900 50  0001 C CNN
+F 3 "" H 3500 1900 50  0001 C CNN
+	1    3500 1900
+	1    0    0    -1
+$EndComp
+$Comp
+L Device:C C1
+U 1 1 5E5E4130
+P 2950 2500
+F 0 "C1" H 3065 2546 50  0000 L CNN
+F 1 "10u" H 3065 2455 50  0000 L CNN
+F 2 "Capacitor_SMD:C_0805_2012Metric_Pad1.15x1.40mm_HandSolder" H 2988 2350 50  0001 C CNN
+F 3 "~" H 2950 2500 50  0001 C CNN
+	1    2950 2500
+	1    0    0    -1
+$EndComp
+Text Label 2850 2750 2    50   ~ 0
+GLV_RTN
+Wire Wire Line
+	2850 2750 2950 2750
+Wire Wire Line
+	2950 2650 2950 2750
+Connection ~ 2950 2750
+Wire Wire Line
+	2950 2350 2950 2250
+Wire Wire Line
+	2950 2250 3150 2250
+Text Label 2850 2250 2    50   ~ 0
+GLV_24V
+Wire Wire Line
+	2850 2250 2950 2250
+Connection ~ 2950 2250
+$Comp
+L Device:C C4
+U 1 1 5E5E78E5
+P 4000 2500
+F 0 "C4" H 4115 2546 50  0000 L CNN
+F 1 "10u" H 4115 2455 50  0000 L CNN
+F 2 "Capacitor_SMD:C_0805_2012Metric_Pad1.15x1.40mm_HandSolder" H 4038 2350 50  0001 C CNN
+F 3 "~" H 4000 2500 50  0001 C CNN
+	1    4000 2500
+	1    0    0    -1
+$EndComp
+Wire Wire Line
+	4000 2750 4000 2650
+Wire Wire Line
+	3850 2250 4000 2250
+Wire Wire Line
+	4000 2250 4000 2350
+Text Label 4100 2250 0    50   ~ 0
+GLV_9V
+Wire Wire Line
+	4100 2250 4000 2250
+Connection ~ 4000 2250
+Wire Wire Line
+	2950 2750 3500 2750
+Wire Wire Line
+	3500 2650 3500 2750
+Connection ~ 3500 2750
+Wire Wire Line
+	3500 2750 4000 2750
+Wire Wire Line
+	4925 4650 4850 4650
+Text Label 4850 4650 2    50   ~ 0
+GLV_RTN
+Wire Wire Line
+	4925 4750 4850 4750
+Text Label 4850 4750 2    50   ~ 0
+GLV_9V
 $EndSCHEMATC

Commit message: added new versions of board
Parts:
- removed C1, C2, C4: 10u, Capacitor_SMD:C_0805_2012Metric_Pad1.15x1.40mm_HandSolder, symbol Device:C
- removed C3: 22u, Capacitor_SMD:C_0805_2012Metric_Pad1.15x1.40mm_HandSolder, symbol Device:C
- removed H1, H2, H3, H4: MountingHole, MountingHole:MountingHole_3.2mm_M3, symbol Mechanical:MountingHole
- removed J1: GLV/CAN, Connector_JST:JST_PH_S4B-PH-SM4-TB_1x04-1MP_P2.00mm_Horizontal, symbol Connector_Generic:Conn_01x04
- removed U2: V7805-500, Lafayette_Electric_Car_Footprints:VX7805-500, symbol Lafayette_Electric_Car_Internals:V7805-500
- removed U3: V7809-500, Lafayette_Electric_Car_Footprints:VX7805-500, symbol Lafayette_Electric_Car_Internals:V7809-500
- added C1, C2: .1u, Capacitor_SMD:C_0805_2012Metric_Pad1.15x1.40mm_HandSolder, symbol pspice:C
- added C3, C4: .33u, Capacitor_SMD:C_0805_2012Metric_Pad1.15x1.40mm_HandSolder, symbol pspice:C
- added H1, H2, H3, H4: MountingHole_Pad, MountingHole:MountingHole_5mm, symbol Mechanical:MountingHole_Pad
- added J1: GLV/CAN, Connector_JST:JST_PH_S6B-PH-SM4-TB_1x06-1MP_P2.00mm_Horizontal, symbol Connector_Generic:Conn_01x06
- added U2: L78L05CD13TR, Package_SO:SO-8_3.9x4.9mm_P1.27mm, symbol Lafayette_Electric_Car_Internals:L78L05CD13TR
- added U3: L78L09CD13TR, Package_SO:SO-8_3.9x4.9mm_P1.27mm, symbol Lafayette_Electric_Car_Internals:L78L09CD13TR
- added U4: 2.9epaper, Lafayette_Electric_Car_Footprints:2.9inEpaper, symbol Lafayette_Electric_Car_Internals:2.9epaper
Connections:
- net labels added: CAN_SHIELD, CH_GND
- wire segments 100 -> 118

Commit message: v4 board
Connections:
- wire segments 118 -> 130
- no-connect marks 1 -> 13
Other:
- moved on the sheet: ESP321
Changed lines of the file:
@@
 L ESP32_Shield-cache:ESP32_Devkit_DOIT_V1 ESP321
 U 1 1 5E39D9F9
-P 5650 4000
-F 0 "ESP321" H 5650 4962 50  0000 C CNN
-F 1 "ESP32_Devkit_DOIT_V1" H 5650 4856 50  0000 C CNN
-F 2 "ESP32_Shield:ESP32_Devkit_DOIT_V1" H 5650 4000 50  0001 C CNN
-F 3 "" H 5650 4000 50  0001 C CNN
-	1    5650 4000
+P 5950 4200
+F 0 "ESP321" H 5950 5162 50  0000 C CNN
+F 1 "ESP32_Devkit_DOIT_V1" H 5950 5056 50  0000 C CNN
+F 2 "ESP32_Shield:ESP32_Devkit_DOIT_V1" H 5950 4200 50  0001 C CNN
+F 3 "" H 5950 4200 50  0001 C CNN
+	1    5950 4200
 	1    0    0    -1
 $EndComp
@@
 ESP_GND
 Wire Wire Line
-	4925 3750 4850 3750
-Text Label 4850 3750 2    50   ~ 0
+	5225 3950 5150 3950
+Text Label 5150 3950 2    50   ~ 0
 ESP_BUTTON2
 Wire Wire Line
-	4925 3650 4850 3650
-Text Label 4850 3650 2    50   ~ 0
+	5225 3850 5150 3850
+Text Label 5150 3850 2    50   ~ 0
 ESP_BUTTON1
 Wire Wire Line
-	4925 4350 4850 4350
-Text Label 4850 4350 2    50   ~ 0
+	5225 4550 5150 4550
+Text Label 5150 4550 2    50   ~ 0
 CLK
 Wire Wire Line
-	4925 4550 4850 4550
-Text Label 4850 4550 2    50   ~ 0
+	5225 4750 5150 4750
+Text Label 5150 4750 2    50   ~ 0
 DIN
 Wire Wire Line
-	6375 3450 6450 3450
-Text Label 6450 3450 0    50   ~ 0
+	6675 3650 6750 3650
+Text Label 6750 3650 0    50   ~ 0
 DC
 Wire Wire Line
-	6375 3750 6450 3750
-Text Label 6450 3750 0    50   ~ 0
+	6675 3950 6750 3950
+Text Label 6750 3950 0    50   ~ 0
 RST
 Wire Wire Line
-	6375 4250 6450 4250
-Text Label 6450 4250 0    50   ~ 0
+	6675 4450 6750 4450
+Text Label 6750 4450 0    50   ~ 0
 BUSY
 Wire Wire Line
-	6375 4550 6450 4550
-Text Label 6450 4550 0    50   ~ 0
+	6675 4750 6750 4750
+Text Label 6750 4750 0    50   ~ 0
 CS
 Wire Wire Line
-	6375 4650 6450 4650
-Text Label 6450 4650 0    50   ~ 0
+	6675 4850 6750 4850
+Text Label 6750 4850 0    50   ~ 0
 ESP_GND
 Wire Wire Line
-	6375 4750 6450 4750
-Text Label 6450 4750 0    50   ~ 0
+	6675 4950 6750 4950
+Text Label 6750 4950 0    50   ~ 0
 ESP_3V3
 Wire Wire Line
-	6375 4450 6450 4450
-Text Label 6450 4450 0    50   ~ 0
+	6675 4650 6750 4650
+Text Label 6750 4650 0    50   ~ 0
 ~R1
 Wire Wire Line
-	6375 4150 6450 4150
-Text Label 6450 4150 0    50   ~ 0
+	6675 4350 6750 4350
+Text Label 6750 4350 0    50   ~ 0
 ~G1
 Wire Wire Line
-	4925 4150 4850 4150
-Text Label 4850 4150 2    50   ~ 0
+	5225 4350 5150 4350
+Text Label 5150 4350 2    50   ~ 0
 ~G2
 Wire Wire Line
-	4925 4050 4850 4050
-Text Label 4850 4050 2    50   ~ 0
+	5225 4250 5150 4250
+Text Label 5150 4250 2    50   ~ 0
 ~R2
 $Comp
@@
 BUTTON2
 Wire Wire Line
-	6375 4350 6450 4350
-Text Label 6450 4350 0    50   ~ 0
+	6675 4550 6750 4550
+Text Label 6750 4550 0    50   ~ 0
 CANTX
 Wire Wire Line
-	6375 4050 6450 4050
-Text Label 6450 4050 0    50   ~ 0
+	6675 4250 6750 4250
+Text Label 6750 4250 0    50   ~ 0
 CANRX
 $Comp
@@
 Do not populate 120ohm resistor. Footprint is left open for debugging.
 Wire Wire Line
-	4925 4650 4850 4650
-Text Label 4850 4650 2    50   ~ 0
+	5225 4850 5150 4850
+Text Label 5150 4850 2    50   ~ 0
 GLV_RTN
 Wire Wire Line
-	4925 4750 4850 4750
-Text Label 4850 4750 2    50   ~ 0
+	5225 4950 5150 4950
+Text Label 5150 4950 2    50   ~ 0
 GLV_9V
 $Comp
@@
 U 1 1 5E78C86E
 P 2550 4300
-F 0 "H3" H 2650 4349 50  0000 L CNN
-F 1 "MountingHole_Pad" H 2650 4258 50  0000 L CNN
+F 0 "H3" H 2650 4349 50  0001 L CNN
+F 1 "MountingHole_Pad" H 2650 4303 50  0000 L CNN
 F 2 "MountingHole:MountingHole_5mm" H 2550 4300 50  0001 C CNN
 F 3 "~" H 2550 4300 50  0001 C CNN
@@
 U 1 1 5E78CFC2
 P 2550 4600
-F 0 "H4" H 2650 4649 50  0000 L CNN
-F 1 "MountingHole_Pad" H 2650 4558 50  0000 L CNN
+F 0 "H4" H 2650 4649 50  0001 L CNN
+F 1 "MountingHole_Pad" H 2650 4603 50  0000 L CNN
 F 2 "MountingHole:MountingHole_5mm" H 2550 4600 50  0001 C CNN
 F 3 "~" H 2550 4600 50  0001 C CNN
@@
 U 1 1 5E792FE8
 P 1650 4300
-F 0 "H1" H 1750 4349 50  0000 L CNN
-F 1 "MountingHole_Pad" H 1750 4258 50  0000 L CNN
+F 0 "H1" H 1750 4349 50  0001 L CNN
+F 1 "MountingHole_Pad" H 1750 4303 50  0000 L CNN
 F 2 "MountingHole:MountingHole_5mm" H 1650 4300 50  0001 C CNN
 F 3 "~" H 1650 4300 50  0001 C CNN
@@
 U 1 1 5E798F46
 P 1650 4600
-F 0 "H2" H 1750 4649 50  0000 L CNN
-F 1 "MountingHole_Pad" H 1750 4558 50  0000 L CNN
+F 0 "H2" H 1750 4649 50  0001 L CNN
+F 1 "MountingHole_Pad" H 1750 4603 50  0000 L CNN
 F 2 "MountingHole:MountingHole_5mm" H 1650 4600 50  0001 C CNN
 F 3 "~" H 1650 4600 50  0001 C CNN
@@
 	1650 4700 2550 4700
 Connection ~ 1650 4700
+Wire Wire Line
+	5225 3550 5150 3550
+Wire Wire Line
+	5225 3650 5150 3650
+Wire Wire Line
+	5225 3750 5150 3750
+Wire Wire Line
+	5225 4050 5150 4050
+Wire Wire Line
+	5225 4150 5150 4150
+Wire Wire Line
+	5225 4450 5150 4450
+Wire Wire Line
+	5225 4650 5150 4650
+Wire Wire Line
+	6675 3550 6750 3550
+Wire Wire Line
+	6675 3750 6750 3750
+Wire Wire Line
+	6675 3850 6750 3850
+Wire Wire Line
+	6675 4050 6750 4050
+Wire Wire Line
+	6675 4150 6750 4150
+NoConn ~ 6750 3550
+NoConn ~ 6750 3750
+NoConn ~ 6750 3850
+NoConn ~ 6750 4050
+NoConn ~ 6750 4150
+NoConn ~ 5150 3550
+NoConn ~ 5150 3650
+NoConn ~ 5150 3750
+NoConn ~ 5150 4050
+NoConn ~ 5150 4150
+NoConn ~ 5150 4450
+NoConn ~ 5150 4650
 $EndSCHEMATC

Commit message: added ams
Parts:
- added J3: Conn_01x02, Connector_JST:JST_PH_S2B-PH-SM4-TB_1x02-1MP_P2.00mm_Horizontal, symbol Connector_Generic:Conn_01x02
- added Q1: BSS84, Package_TO_SOT_SMD:SOT-23, symbol Transistor_FET:BSS84
- added Q?: BSS138W, Package_TO_SOT_SMD:SOT-323_SC-70_Handsoldering, symbol Lafayette_Electric_Car_Internals:BSS138W
- added R1: 0, Resistor_SMD:R_0805_2012Metric_Pad1.15x1.40mm_HandSolder, symbol Device:R
- added R?: 2.4K, Resistor_SMD:R_0805_2012Metric_Pad1.15x1.40mm_HandSolder, symbol Device:R
- added R?: 7.5K, Resistor_SMD:R_0805_2012Metric_Pad1.15x1.40mm_HandSolder, symbol Device:R
Connections:
- net labels added: AMS_FLT, AMS_FLT_LED, GLV_24
- wire segments 130 -> 142
- no-connect marks 13 -> 12
Changed lines of the file:
@@
 Wire Wire Line
 	6675 4250 6750 4250
-Text Label 6750 4250 0    50   ~ 0
-CANRX
 $Comp
 L Device:R R3
@@
 Wire Wire Line
 	6675 3850 6750 3850
-Wire Wire Line
-	6675 4050 6750 4050
-Wire Wire Line
-	6675 4150 6750 4150
 NoConn ~ 6750 3550
 NoConn ~ 6750 3750
 NoConn ~ 6750 3850
-NoConn ~ 6750 4050
-NoConn ~ 6750 4150
 NoConn ~ 5150 3550
 NoConn ~ 5150 3650
@@
 NoConn ~ 5150 4450
 NoConn ~ 5150 4650
+Text Label 6750 4150 0    50   ~ 0
+AMS_FLT
+NoConn ~ 6750 4050
+Wire Wire Line
+	6675 4150 6750 4150
+Wire Wire Line
+	6675 4050 6750 4050
+Text Label 6750 4250 0    50   ~ 0
+CANRX
+$Comp
+L Connector_Generic:Conn_01x02 J3
+U 1 1 5E6E9855
+P 5150 7000
+F 0 "J3" H 5230 6992 50  0000 L CNN
+F 1 "Conn_01x02" H 5230 6901 50  0000 L CNN
+F 2 "Connector_JST:JST_PH_S2B-PH-SM4-TB_1x02-1MP_P2.00mm_Horizontal" H 5150 7000 50  0001 C CNN
+F 3 "~" H 5150 7000 50  0001 C CNN
+	1    5150 7000
+	1    0    0    -1
+$EndComp
+Wire Wire Line
+	4950 7000 4800 7000
+Text Label 4800 7000 2    50   ~ 0
+AMS_FLT_LED
+Wire Wire Line
+	4950 7100 4800 7100
+Text Label 4800 7100 2    50   ~ 0
+GLV_RTN
+Text Label 1000 7450 2    50   ~ 0
+AMS_FLT
+Wire Wire Line
+	1100 7450 1000 7450
+Text Label 1400 6250 0    50   ~ 0
+GLV_24
+Wire Wire Line
+	1400 6400 1400 6250
+Wire Wire Line
+	1400 6800 1400 6700
+Connection ~ 1400 6800
+Wire Wire Line
+	1550 6800 1400 6800
+Wire Wire Line
+	1400 6950 1400 6800
+$Comp
+L Device:R R?
+U 1 1 5E72A72B
+P 1400 7100
+F 0 "R?" H 1470 7146 50  0000 L CNN
+F 1 "7.5K" H 1470 7055 50  0000 L CNN
+F 2 "Resistor_SMD:R_0805_2012Metric_Pad1.15x1.40mm_HandSolder" V 1330 7100 50  0001 C CNN
+F 3 "~" H 1400 7100 50  0001 C CNN
+	1    1400 7100
+	1    0    0    -1
+$EndComp
+$Comp
+L Device:R R?
+U 1 1 5E722263
+P 1400 6550
+F 0 "R?" H 1470 6596 50  0000 L CNN
+F 1 "2.4K" H 1470 6505 50  0000 L CNN
+F 2 "Resistor_SMD:R_0805_2012Metric_Pad1.15x1.40mm_HandSolder" V 1330 6550 50  0001 C CNN
+F 3 "~" H 1400 6550 50  0001 C CNN
+	1    1400 6550
+	1    0    0    -1
+$EndComp
+Text Label 2400 7100 0    50   ~ 0
+AMS_FLT_LED
+Wire Wire Line
+	2250 7100 2400 7100
+$Comp
+L Device:R R1
+U 1 1 5E6DEC6F
+P 2100 7100
+F 0 "R1" V 1893 7100 50  0000 C CNN
+F 1 "0" V 1984 7100 50  0000 C CNN
+F 2 "Resistor_SMD:R_0805_2012Metric_Pad1.15x1.40mm_HandSolder" V 2030 7100 50  0001 C CNN
+F 3 "~" H 2100 7100 50  0001 C CNN
+	1    2100 7100
+	0    1    1    0
+$EndComp
+Wire Wire Line
+	1850 7100 1950 7100
+Wire Wire Line
+	1850 7000 1850 7100
+Text Label 1850 6500 0    50   ~ 0
+GLV_24V
+Wire Wire Line
+	1850 6600 1850 6500
+$Comp
+L Transistor_FET:BSS84 Q1
+U 1 1 5E694329
+P 1750 6800
+F 0 "Q1" H 1956 6846 50  0000 L CNN
+F 1 "BSS84" H 1956 6755 50  0000 L CNN
+F 2 "Package_TO_SOT_SMD:SOT-23" H 1950 6725 50  0001 L CIN
+F 3 "http://assets.nexperia.com/documents/data-sheet/BSS84.pdf" H 1750 6800 50  0001 L CNN
+	1    1750 6800
+	1    0    0    1
+$EndComp
+$Comp
+L Lafayette_Electric_Car_Internals:BSS138W Q?
+U 1 1 5E76FF66
+P 1400 7450
+F 0 "Q?" H 1506 7496 50  0000 L CNN
+F 1 "BSS138W" H 1506 7405 50  0000 L CNN
+F 2 "Package_TO_SOT_SMD:SOT-323_SC-70_Handsoldering" H 1100 7950 50  0001 C CNN
+F 3 "https://www.mouser.com/datasheet/2/308/BSS138W-1305267.pdf" H 1400 7450 50  0001 C CNN
+F 4 "BSS138WH6327XTSA1CT-ND" H 800 7850 50  0001 C CNN "Vendor Part"
+F 5 "Digikey" H 1400 7450 50  0001 C CNN "Vendor"
+F 6 "Infineon Technologies" H 1400 7450 50  0001 C CNN "Manufacturer"
+F 7 "BSS138WH6327XTSA1" H 1400 7450 50  0001 C CNN "Manufacturer Part"
+	1    1400 7450
+	1    0    0    -1
+$EndComp
+Wire Wire Line
+	1400 7650 1400 7800
+Text Label 1400 7800 0    50   ~ 0
+GLV_RTN
 $EndSCHEMATC
