File: Leah/DriverDisplay5.kicad_pcb (KiCad board)
At the start: 2 copper layers, 126.8 x 42.3 mm, 40 parts, among them J1 GLV/CAN, J2 Display, J3 Conn_01x02, Q1 BSS84, Q2 BSS138W, U1 MCP2551-I-SN, U2 L78L05CD13TR, U3 L78L09CD13TR, U4 2.9epaper

Commit message: added ams
Parts:
- removed J3: Conn_01x02, Connector_JST:JST_PH_S2B-PH-SM4-TB_1x02-1MP_P2.00mm_Horizontal
- removed Q1: BSS84, Package_TO_SOT_SMD:SOT-23
- removed Q2: BSS138W, Package_TO_SOT_SMD:SOT-323_SC-70_Handsoldering
- removed R1: 0, Resistor_SMD:R_0805_2012Metric_Pad1.15x1.40mm_HandSolder
- removed R12: 2.4K, Resistor_SMD:R_0805_2012Metric_Pad1.15x1.40mm_HandSolder
- removed R13: 7.5K, Resistor_SMD:R_0805_2012Metric_Pad1.15x1.40mm_HandSolder
Connections:
- ESP321 pad 24: /AMS_FLT -> Net-(ESP321-Pad24)
Routing:
- net /AMS_FLT: track 61.9 -> 0.00 mm, vias 4 -> 0
- net /GLV_24V: track 79.5 -> 57.4 mm
- net Net-(Q1-Pad1): track 21.7 -> 0.00 mm
- net /AMS_FLT_LED: track 9.77 -> 0.00 mm
- net Net-(Q2-Pad3): track 7.99 -> 0.00 mm
- net Net-(Q1-Pad3): track 6.47 -> 0.00 mm
- net /DC: track 57.1 -> 60.1 mm
- net /GLV_RTN: track 141.3 -> 140.7 mm
